File: device_decoder.kicad_sch (KiCad schematic)
At the start: 9 parts, among them U22 74LS04, U24 74LS10, U29 74LS20, U5 74LS138, U6 74LS138, U8 74LS30

Commit message: finished routing rev3
Changed lines of the file:
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@@
 	)
 	(hierarchical_label "~{RTC CS}"
-		(shape input)
+		(shape output)
 		(at 208.28 53.34 0)
 		(effects
@@
 	)
 	(hierarchical_label "~{DMA CS}"
-		(shape input)
+		(shape output)
 		(at 208.28 31.75 0)
 		(effects
@@
 	)
 	(hierarchical_label "~{UART CS}"
-		(shape input)
+		(shape output)
 		(at 208.28 49.53 0)
 		(effects
@@
 	)
 	(hierarchical_label "~{PPI CS}"
-		(shape input)
+		(shape output)
 		(at 208.28 46.99 0)
 		(effects
@@
 	)
 	(hierarchical_label "~{DMA REG CS}"
-		(shape input)
+		(shape output)
 		(at 208.28 41.91 0)
 		(effects
@@
 	)
 	(hierarchical_label "~{FLAG CS}"
-		(shape input)
+		(shape output)
 		(at 208.28 44.45 0)
 		(effects
@@
 	)
 	(hierarchical_label "~{PIT CS}"
-		(shape input)
+		(shape output)
 		(at 208.28 36.83 0)
 		(effects
@@
 	)
 	(hierarchical_label "~{KBRD CS}"
-		(shape input)
+		(shape output)
 		(at 208.28 39.37 0)
 		(effects

Commit message: fixed things
Connections:
- net +5V: now also U24.4, U24.5, U8.11, U8.6; no longer U8.2, U8.3
- net XA9: no longer U24.4, U24.5
- net ~{RAM_BANK_CS}: now also U6.11 (O4), U8.5; no longer U6.12 (O3), U8.4
- net ~{ROM_CS}: now also U6.7 (O7), U8.12; no longer U6.15 (O0), U8.1
- net at U6.13 (O2): now also U29.12, U8.3
- net at U6.14 (O1): now also U29.10, U8.2
- new net: U29.9, U6.15 (O0), U8.1
- new net: U29.13, U6.12 (O3), U8.4
- now unconnected: U6.10 (O5), U6.9 (O6)
Other:
- note added: "IO MAP 000-01F : DMA 020-03F : PIC 040-05F : PIT 060-07F : KBRD 080-09F : DMA REG 0A0-0BF : FLAG 0CF-0DF : PPI 0E0-0FF : UART 100-1FF : RTC 200-3FF : ISA BUS I/O"
- note added: "MEM MAP E0000-FFFFF: ROM D0000-DFFFF: Expansion Card 1 C0000-CFFFF: Expansion Card 1 B0000-BFFFF: Monochrome Video A0000-AFFFF: Color Memory 80000-9FFFF: BANKED RAM 00000-7FFFF: RAM"
- note removed: "IO MAP 000-01F : DMA 020-03F : PIC 040-05F : PIT 060-07F : KBRD 080-09F : DMA REG 0A0-0BF : FLAG 0CF-0DF : PPI 0E0-0FF : UART 100-1FF : RTC"
- note removed: "MEM MAP E0000-FFFFF: ROM D0000-DFFFF: Expansion Card 1 C0000-CFFFF: Expansion Card 1 B0000-BFFFF: Monochrome Video A0000-AFFFF: Color Memory 00000-9FFFF: RAM"

Commit message: Upgraded speaker, esd protection, added dip sockets, adjusted routing
Parts:
- U22, U24, U29, U8: footprint Package_DIP:DIP-14_W7.62mm -> Package_DIP:DIP-14_W7.62mm_Socket
- U5, U6: footprint Package_DIP:DIP-16_W7.62mm -> Package_DIP:DIP-16_W7.62mm_Socket
Other:
- note added: "~AEN & XA8 & ~XA9"
- note added: "~AEN & ~XA8 & ~XA9"
Changed lines of the file:
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@@
 		)
 	)
+	(text "~AEN & XA8 & ~XA9"
+		(exclude_from_sim no)
+		(at 92.456 67.818 0)
+		(effects
+			(font
+				(size 1.27 1.27)
+			)
+		)
+	)
 	(text "MEMORY MAP"
 		(exclude_from_sim no)
@@
 		)
 	)
+	(text "~AEN & ~XA8 & ~XA9"
+		(exclude_from_sim no)
+		(at 92.71 39.878 0)
+		(effects
+			(font
+				(size 1.27 1.27)
+			)
+		)
+	)
 	(text "IO MAP\n000-01F : DMA\n020-03F : PIC\n040-05F : PIT\n060-07F : KBRD\n080-09F : DMA REG\n0A0-0BF : FLAG\n0CF-0DF : PPI\n0E0-0FF : UART\n100-1FF : RTC\n200-3FF : ISA BUS I/O"
 		(exclude_from_sim no)
@@
 	(bus
 		(pts
-			(xy 88.9 25.4) (xy 109.22 25.4)
+			(xy 93.98 25.4) (xy 109.22 25.4)
 		)
 		(stroke
@@
 	(wire
 		(pts
-			(xy 97.79 44.45) (xy 105.41 44.45)
+			(xy 93.98 44.45) (xy 105.41 44.45)
 		)
 		(stroke
@@
 		)
 	)
-	(label "XA[19..0]"
+	(label "XA[9..0]"
 		(at 97.79 25.4 0)
 		(effects
@@
 	(hierarchical_label "XA[9..0]"
 		(shape input)
-		(at 88.9 25.4 180)
+		(at 93.98 25.4 180)
 		(effects
 			(font
@@
 	(hierarchical_label "~{AEN}"
 		(shape input)
-		(at 97.79 44.45 180)
+		(at 93.98 44.45 180)
 		(effects
 			(font
@@
 			)
 		)
-		(property "Footprint" "Package_DIP:DIP-14_W7.62mm"
+		(property "Footprint" "Package_DIP:DIP-14_W7.62mm_Socket"
 			(at 26.67 176.53 0)
 			(hide yes)
@@
 			)
 		)
+		(property "Sim.Device" ""
+			(at 26.67 176.53 0)
+			(hide yes)
+			(show_name no)
+			(do_not_autoplace no)
+			(effects
+				(font
+					(size 1.27 1.27)
+				)
+			)
+		)
 		(pin "5"
 		)
@@
 			)
 		)
+		(property "Sim.Device" ""
+			(at 107.95 180.34 0)
+			(hide yes)
+			(show_name no)
+			(do_not_autoplace no)
+			(effects
+				(font
+					(size 1.27 1.27)
+				)
+			)
+		)
 		(pin "2"
 		)
@@
 			)
 		)
+		(property "Sim.Device" ""
+			(at 80.01 180.34 0)
+			(hide yes)
+			(show_name no)
+			(do_not_autoplace no)
+			(effects
+				(font
+					(size 1.27 1.27)
+				)
+			)
+		)
 		(pin "2"
 		)
@@
 			)
 		)
-		(property "Footprint" "Package_DIP:DIP-14_W7.62mm"
+		(property "Footprint" "Package_DIP:DIP-14_W7.62mm_Socket"
 			(at 180.34 151.13 0)
 			(hide yes)
@@
 			)
 		)
+		(property "Sim.Device" ""
+			(at 180.34 151.13 0)
+			(hide yes)
+			(show_name no)
+			(do_not_autoplace no)
+			(effects
+				(font
+					(size 1.27 1.27)
+				)
+			)
+		)
 		(pin "3"
 		)
@@
 			)
 		)
-		(property "Footprint" "Package_DIP:DIP-16_W7.62mm"
+		(property "Footprint" "Package_DIP:DIP-16_W7.62mm_Socket"
 			(at 133.35 39.37 0)
 			(hide yes)
@@
 			)
 		)
+		(property "Sim.Device" ""
+			(at 133.35 39.37 0)
+			(hide yes)
+			(show_name no)
+			(do_not_autoplace no)
+			(effects
+				(font
+					(size 1.27 1.27)
+				)
+			)
+		)
 		(pin "14"
 		)
@@
 			)
 		)
-		(property "Footprint" "Package_DIP:DIP-14_W7.62mm"
+		(property "Footprint" "Package_DIP:DIP-14_W7.62mm_Socket"
 			(at 160.02 119.38 0)
 			(hide yes)
@@
 			)
 		)
+		(property "Sim.Device" ""
+			(at 160.02 119.38 0)
+			(hide yes)
+			(show_name no)
+			(do_not_autoplace no)
+			(effects
+				(font
+					(size 1.27 1.27)
+				)
+			)
+		)
 		(pin "5"
 		)
@@
 			)
 		)
-		(property "Footprint" "Package_DIP:DIP-14_W7.62mm"
+		(property "Footprint" "Package_DIP:DIP-14_W7.62mm_Socket"
 			(at 180.34 119.38 0)
 			(hide yes)
@@
 			)
 		)
+		(property "Sim.Device" ""
+			(at 180.34 119.38 0)
+			(hide yes)
+			(show_name no)
+			(do_not_autoplace no)
+			(effects
+				(font
+					(size 1.27 1.27)
+				)
+			)
+		)
 		(pin "3"
 		)
@@
 			)
 		)
+		(property "Sim.Device" ""
+			(at 93.98 180.34 0)
+			(hide yes)
+			(show_name no)
+			(do_not_autoplace no)
+			(effects
+				(font
+					(size 1.27 1.27)
+				)
+			)
+		)
 		(pin "2"
 		)
@@
 			)
 		)
-		(property "Footprint" "Package_DIP:DIP-16_W7.62mm"
+		(property "Footprint" "Package_DIP:DIP-16_W7.62mm_Socket"
 			(at 113.03 119.38 0)
 			(hide yes)
@@
 			)
 		)
+		(property "Sim.Device" ""
+			(at 113.03 119.38 0)
+			(hide yes)
+			(show_name no)
+			(do_not_autoplace no)
+			(effects
+				(font
+					(size 1.27 1.27)
+				)
+			)
+		)
 		(pin "14"
 		)
@@
 			)
 		)
-		(property "Footprint" "Package_DIP:DIP-14_W7.62mm"
+		(property "Footprint" "Package_DIP:DIP-14_W7.62mm_Socket"
 			(at 142.24 80.01 0)
 			(hide yes)
@@
 			)
 		)
+		(property "Sim.Device" ""
+			(at 142.24 80.01 0)
+			(hide yes)
+			(show_name no)
+			(do_not_autoplace no)
+			(effects
+				(font
+					(size 1.27 1.27)
+				)
+			)
+		)
 		(pin "8"
 		)
@@
 			)
 		)
-		(property "Footprint" "Package_DIP:DIP-14_W7.62mm"
+		(property "Footprint" "Package_DIP:DIP-14_W7.62mm_Socket"
 			(at 170.18 68.58 0)
 			(hide yes)
@@
 			)
 		)
+		(property "Sim.Device" ""
+			(at 170.18 68.58 0)
+			(hide yes)
+			(show_name no)
+			(do_not_autoplace no)
+			(effects
+				(font
+					(size 1.27 1.27)
+				)
+			)
+		)
 		(pin "8"
 		)
@@
 			)
 		)
-		(property "Footprint" "Package_DIP:DIP-14_W7.62mm"
+		(property "Footprint" "Package_DIP:DIP-14_W7.62mm_Socket"
 			(at 160.02 151.13 0)
 			(hide yes)
@@
 			(at 160.02 151.13 0)
 			(hide yes)
+			(show_name no)
+			(do_not_autoplace no)
+			(effects
+				(font
+					(size 1.27 1.27)
+				)
+			)
+		)
+		(property "Sim.Device" ""
+			(at 160.02 151.13 0)
+			(hide yes)

Commit message: final commit before spinning
Changed lines of the file:
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@@
 	)
 	(hierarchical_label "XA[9..0]"
-		(shape input)
+		(shape tri_state)
 		(at 93.98 25.4 180)
 		(effects
