File: flag_registers.kicad_sch (KiCad schematic)
At the start: 8 parts, among them U17 74LS32, U54 74LS273, U55 74LS244

Commit message: Progress routing
Connections:
- net +5V: now also U17.14 (VCC)
Changed lines of the file:
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@@
 	(symbol
 		(lib_id "power:VCC")
-		(at 245.11 48.26 0)
+		(at 243.84 48.26 0)
 		(unit 1)
 		(body_style 1)
@@
 		(fields_autoplaced yes)
 		(property "Reference" "#PWR0205"
-			(at 245.11 52.07 0)
+			(at 243.84 52.07 0)
 			(hide yes)
 			(show_name no)
@@
 		)
 		(property "Value" "+5V"
-			(at 245.11 43.18 0)
+			(at 243.84 43.18 0)
 			(show_name no)
 			(do_not_autoplace no)
@@
 		)
 		(property "Footprint" ""
-			(at 245.11 48.26 0)
+			(at 243.84 48.26 0)
 			(hide yes)
 			(show_name no)
@@
 		)
 		(property "Datasheet" ""
-			(at 245.11 48.26 0)
+			(at 243.84 48.26 0)
 			(hide yes)
 			(show_name no)
@@
 		)
 		(property "Description" "Power symbol creates a global label with name \"VCC\""
-			(at 245.11 48.26 0)
+			(at 243.84 48.26 0)
 			(hide yes)
 			(show_name no)

Commit message: fixed things
Changed lines of the file:
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@@
 	)
 	(hierarchical_label "SPKR EN"
-		(shape input)
+		(shape output)
 		(at 205.74 55.88 0)
 		(effects
@@
 	)
 	(hierarchical_label "SPKR GATE"
-		(shape input)
+		(shape output)
 		(at 205.74 58.42 0)
 		(effects

Commit message: Upgraded speaker, esd protection, added dip sockets, adjusted routing
Parts:
- U17: footprint Package_DIP:DIP-14_W7.62mm -> Package_DIP:DIP-14_W7.62mm_Socket
- U54, U55: footprint Package_DIP:DIP-20_W7.62mm -> Package_DIP:DIP-20_W7.62mm_Socket
Connections:
- net GND: no longer U55.19 (OEb)
- net at U17.11, U55.1 (OEa): now also U55.19 (OEb)
Other:
- moved on the sheet: U17E
Changed lines of the file:
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@@
 	)
 	(junction
-		(at 142.24 138.43)
-		(diameter 0)
-		(color 0 0 0 0)
-	)
-	(junction
 		(at 176.53 66.04)
 		(diameter 0)
@@
 	)
 	(junction
+		(at 160.02 129.54)
+		(diameter 0)
+		(color 0 0 0 0)
+	)
+	(junction
 		(at 163.83 53.34)
 		(diameter 0)
@@
 	(wire
 		(pts
-			(xy 142.24 138.43) (xy 157.48 138.43)
-		)
-		(stroke
-			(width 0)
-			(type default)
-		)
-	)
-	(wire
-		(pts
 			(xy 154.94 104.14) (xy 161.29 104.14)
 		)
@@
 	(wire
 		(pts
-			(xy 142.24 137.16) (xy 142.24 138.43)
-		)
-		(stroke
-			(width 0)
-			(type default)
-		)
-	)
-	(wire
-		(pts
 			(xy 69.85 71.12) (xy 69.85 90.17)
 		)
@@
 	(wire
 		(pts
-			(xy 157.48 129.54) (xy 154.94 129.54)
+			(xy 154.94 68.58) (xy 179.07 68.58)
 		)
 		(stroke
@@
 		)
 	)
-	(wire
+	(bus
 		(pts
-			(xy 154.94 68.58) (xy 179.07 68.58)
+			(xy 186.69 53.34) (xy 205.74 53.34)
 		)
 		(stroke
@@
 		)
 	)
-	(bus
+	(wire
 		(pts
-			(xy 186.69 53.34) (xy 205.74 53.34)
+			(xy 123.19 63.5) (xy 129.54 63.5)
 		)
 		(stroke
@@
 	(wire
 		(pts
-			(xy 123.19 63.5) (xy 129.54 63.5)
+			(xy 160.02 129.54) (xy 160.02 127)
 		)
 		(stroke
@@
 	(wire
 		(pts
-			(xy 142.24 138.43) (xy 142.24 139.7)
+			(xy 142.24 137.16) (xy 142.24 139.7)
 		)
 		(stroke
@@
 	(wire
 		(pts
-			(xy 123.19 58.42) (xy 129.54 58.42)
+			(xy 154.94 129.54) (xy 160.02 129.54)
 		)
 		(stroke
@@
 	(wire
 		(pts
-			(xy 171.45 60.96) (xy 205.74 60.96)
+			(xy 123.19 58.42) (xy 129.54 58.42)
 		)
 		(stroke
@@
 	(wire
 		(pts
-			(xy 157.48 138.43) (xy 157.48 129.54)
+			(xy 171.45 60.96) (xy 205.74 60.96)
 		)
 		(stroke
@@
 	(wire
 		(pts
-			(xy 160.02 149.86) (xy 160.02 127)
+			(xy 160.02 149.86) (xy 160.02 129.54)
 		)
 		(stroke
@@
 			)
 		)
+		(property "Sim.Device" ""
+			(at 213.36 25.4 0)
+			(hide yes)
+			(show_name no)
+			(do_not_autoplace no)
+			(effects
+				(font
+					(size 1.27 1.27)
+				)
+			)
+		)
 		(pin "2"
 		)
@@
 			)
 		)
+		(property "Sim.Device" ""
+			(at 257.81 25.4 0)
+			(hide yes)
+			(show_name no)
+			(do_not_autoplace no)
+			(effects
+				(font
+					(size 1.27 1.27)
+				)
+			)
+		)
 		(pin "2"
 		)
@@
 			)
 		)
-		(property "Footprint" "Package_DIP:DIP-14_W7.62mm"
+		(property "Footprint" "Package_DIP:DIP-14_W7.62mm_Socket"
 			(at 88.9 73.66 0)
 			(hide yes)
@@
 			)
 		)
+		(property "Sim.Device" ""
+			(at 88.9 73.66 0)
+			(hide yes)
+			(show_name no)
+			(do_not_autoplace no)
+			(effects
+				(font
+					(size 1.27 1.27)
+				)
+			)
+		)
 		(pin "7"
 		)
@@
 			)
 		)
-		(property "Footprint" "Package_DIP:DIP-20_W7.62mm"
+		(property "Footprint" "Package_DIP:DIP-20_W7.62mm_Socket"
 			(at 142.24 63.5 0)
 			(hide yes)
@@
 			)
 		)
+		(property "Sim.Device" ""
+			(at 142.24 63.5 0)
+			(hide yes)
+			(show_name no)
+			(do_not_autoplace no)
+			(effects
+				(font
+					(size 1.27 1.27)
+				)
+			)
+		)
 		(pin "14"
 		)
@@
 			)
 		)
-		(property "Footprint" "Package_DIP:DIP-20_W7.62mm"
+		(property "Footprint" "Package_DIP:DIP-20_W7.62mm_Socket"
 			(at 142.24 116.84 0)
 			(hide yes)
@@
 			)
 		)
+		(property "Sim.Device" ""
+			(at 142.24 116.84 0)
+			(hide yes)
+			(show_name no)
+			(do_not_autoplace no)
+			(effects
+				(font
+					(size 1.27 1.27)
+				)
+			)
+		)
 		(pin "19"
 		)
@@
 	(symbol
 		(lib_id "74xx:74LS32")
-		(at 243.84 60.96 0)
+		(at 265.43 59.69 0)
 		(unit 5)
 		(body_style 1)
@@
 		(fields_autoplaced yes)
 		(property "Reference" "U17"
-			(at 250.19 59.6899 0)
+			(at 271.78 58.4199 0)
 			(show_name no)
 			(do_not_autoplace no)
@@
 		)
 		(property "Value" "74LS32"
-			(at 250.19 62.2299 0)
+			(at 271.78 60.9599 0)
 			(show_name no)
 			(do_not_autoplace no)
@@
 			)
 		)
-		(property "Footprint" "Package_DIP:DIP-14_W7.62mm"
-			(at 243.84 60.96 0)
+		(property "Footprint" "Package_DIP:DIP-14_W7.62mm_Socket"
+			(at 265.43 59.69 0)
 			(hide yes)
 			(show_name no)
@@
 		)
 		(property "Datasheet" "http://www.ti.com/lit/gpn/sn74LS32"
-			(at 243.84 60.96 0)
+			(at 265.43 59.69 0)
 			(hide yes)
 			(show_name no)
@@
 		)
 		(property "Description" "Quad 2-input OR"
-			(at 243.84 60.96 0)
+			(at 265.43 59.69 0)
+			(hide yes)
+			(show_name no)
+			(do_not_autoplace no)
+			(effects
+				(font
+					(size 1.27 1.27)
+				)
+			)
+		)
+		(property "Sim.Device" ""
+			(at 265.43 59.69 0)
 			(hide yes)
 			(show_name no)
@@
 	(symbol
 		(lib_id "power:VCC")
-		(at 243.84 48.26 0)
+		(at 265.43 46.99 0)
 		(unit 1)
 		(body_style 1)
@@
 		(fields_autoplaced yes)
 		(property "Reference" "#PWR0205"
-			(at 243.84 52.07 0)
+			(at 265.43 50.8 0)
 			(hide yes)
 			(show_name no)
@@
 		)
 		(property "Value" "+5V"
-			(at 243.84 43.18 0)
+			(at 265.43 41.91 0)
 			(show_name no)
 			(do_not_autoplace no)
@@
 		)
 		(property "Footprint" ""
-			(at 243.84 48.26 0)
+			(at 265.43 46.99 0)
 			(hide yes)
 			(show_name no)
@@
 		)
 		(property "Datasheet" ""
-			(at 243.84 48.26 0)
+			(at 265.43 46.99 0)
 			(hide yes)
 			(show_name no)
@@
 		)
 		(property "Description" "Power symbol creates a global label with name \"VCC\""
-			(at 243.84 48.26 0)
+			(at 265.43 46.99 0)
 			(hide yes)
 			(show_name no)
@@
 			)
 		)
+		(property "Sim.Device" ""
+			(at 242.57 25.4 0)
+			(hide yes)
+			(show_name no)
+			(do_not_autoplace no)
+			(effects
+				(font
+					(size 1.27 1.27)
+				)
+			)
+		)
 		(pin "2"
 		)
@@
 			)
 		)
+		(property "Sim.Device" ""
+			(at 228.6 25.4 0)
+			(hide yes)
+			(show_name no)
+			(do_not_autoplace no)
+			(effects
+				(font
+					(size 1.27 1.27)
+				)
+			)
+		)
 		(pin "2"
 		)
@@
 	(symbol
 		(lib_id "power:GND")
-		(at 243.84 73.66 0)
+		(at 265.43 72.39 0)
 		(unit 1)
 		(body_style 1)
@@
 		(fields_autoplaced yes)
 		(property "Reference" "#PWR0212"
-			(at 243.84 80.01 0)
+			(at 265.43 78.74 0)
 			(hide yes)
 			(show_name no)
@@
 		)
 		(property "Value" "GND"
-			(at 243.84 78.74 0)
+			(at 265.43 77.47 0)
 			(show_name no)
 			(do_not_autoplace no)
@@
 		)
 		(property "Footprint" ""
-			(at 243.84 73.66 0)
+			(at 265.43 72.39 0)
 			(hide yes)
 			(show_name no)
@@
 		)
 		(property "Datasheet" ""
-			(at 243.84 73.66 0)
+			(at 265.43 72.39 0)
 			(hide yes)
 			(show_name no)
@@
 		)
 		(property "Description" "Power symbol creates a global label with name \"GND\" , ground"
-			(at 243.84 73.66 0)
+			(at 265.43 72.39 0)
 			(hide yes)
 			(show_name no)
@@
 			)
 		)
+		(property "Sim.Device" ""
+			(at 271.78 25.4 0)
+			(hide yes)
+			(show_name no)
+			(do_not_autoplace no)
+			(effects
+				(font
+					(size 1.27 1.27)
+				)
+			)
+		)
 		(pin "2"
 		)
@@
 			)
 		)
-		(property "Footprint" "Package_DIP:DIP-14_W7.62mm"
+		(property "Footprint" "Package_DIP:DIP-14_W7.62mm_Socket"
 			(at 88.9 92.71 0)
 			(hide yes)
@@
 			(at 88.9 92.71 0)
 			(hide yes)
+			(show_name no)
+			(do_not_autoplace no)
+			(effects
+				(font
+					(size 1.27 1.27)
+				)
+			)
+		)
+		(property "Sim.Device" ""
+			(at 88.9 92.71 0)
+			(hide yes)

Commit message: final commit before spinning
Changed lines of the file:
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@@
 	)
 	(hierarchical_label "ALLOW NMI"
-		(shape input)
+		(shape output)
 		(at 205.74 68.58 0)
 		(effects
@@
 	)
 	(hierarchical_label "ENABLE IO CK"
-		(shape input)
+		(shape output)
 		(at 205.74 66.04 0)
 		(effects
