File: pinout.kicad_sch (KiCad schematic)
At the start: 1 part, among them J7 Conn_02x14_Odd_Even

Commit message: Upgraded speaker, esd protection, added dip sockets, adjusted routing
Parts:
- added U44: USBLC6-2SC6, Package_TO_SOT_SMD:SOT-23-6, symbol Power_Protection:USBLC6-2SC6
Connections:
- net GND: now also U44.2 (GND)
- net PIT GATE: now also U44.1 (I/O1); no longer J7.28 (Pin_28)
- net PIT OUT: now also U44.3 (I/O2); no longer J7.27 (Pin_27)
- new net: J7.27 (Pin_27), U44.4 (I/O2)
- new net: J7.28 (Pin_28), U44.6 (I/O1)
- new net VCC: U44.5 (VBUS)

Commit message: adjustments to routing
Connections:
- net VCC is gone; now on net +5V: U44.5 (VBUS)
Changed lines of the file:
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@@
 		(dnp no)
 		(fields_autoplaced yes)
-		(property "Reference" "#PWR02"
+		(property "Reference" "#PWR0283"
 			(at 59.69 91.44 0)
 			(hide yes)
@@
 			)
 		)
-		(property "Value" "VCC"
+		(property "Value" "+5V"
 			(at 59.69 82.55 0)
 			(show_name no)
@@
 			(project "retroslop"
 				(path "/c091a5a9-cc18-4de7-90b1-5162a376bd78/94e99637-776f-46be-ad0c-ed4362e4c890"
-					(reference "#PWR02")
+					(reference "#PWR0283")
 					(unit 1)
 				)

Commit message: final commit before spinning
Connections:
- net PIT GATE: now also U44.3 (I/O2); no longer U44.1 (I/O1)
- net PIT OUT: now also U44.1 (I/O1); no longer U44.3 (I/O2)
- net at J7.27 (Pin_27): now also U44.6 (I/O1); no longer U44.4 (I/O2)
- net at J7.28 (Pin_28): now also U44.4 (I/O2); no longer U44.6 (I/O1)
Changed lines of the file:
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@@
-	(wire
-		(pts
-			(xy 90.17 85.09) (xy 99.06 85.09)
-		)
-		(stroke
-			(width 0)
-			(type default)
-		)
-	)
 	(wire
 		(pts
@@
 	(wire
 		(pts
+			(xy 114.3 95.25) (xy 114.3 85.09)
+		)
+		(stroke
+			(width 0)
+			(type default)
+		)
+	)
+	(wire
+		(pts
 			(xy 87.63 69.85) (xy 99.06 69.85)
 		)
@@
 	(wire
 		(pts
+			(xy 93.98 92.71) (xy 93.98 85.09)
+		)
+		(stroke
+			(width 0)
+			(type default)
+		)
+	)
+	(wire
+		(pts
 			(xy 44.45 95.25) (xy 54.61 95.25)
 		)
@@
 	(wire
 		(pts
-			(xy 64.77 95.25) (xy 90.17 95.25)
-		)
-		(stroke
-			(width 0)
-			(type default)
-		)
-	)
-	(wire
-		(pts
-			(xy 64.77 92.71) (xy 115.57 92.71)
+			(xy 64.77 95.25) (xy 114.3 95.25)
 		)
 		(stroke
@@
 	(wire
 		(pts
-			(xy 90.17 95.25) (xy 90.17 85.09)
-		)
-		(stroke
-			(width 0)
-			(type default)
-		)
-	)
-	(wire
-		(pts
 			(xy 78.74 52.07) (xy 99.06 52.07)
 		)
@@
 	(wire
 		(pts
-			(xy 115.57 85.09) (xy 111.76 85.09)
-		)
-		(stroke
-			(width 0)
-			(type default)
-		)
-	)
-	(wire
-		(pts
 			(xy 123.19 74.93) (xy 111.76 74.93)
 		)
@@
 	(wire
 		(pts
+			(xy 111.76 85.09) (xy 114.3 85.09)
+		)
+		(stroke
+			(width 0)
+			(type default)
+		)
+	)
+	(wire
+		(pts
 			(xy 111.76 52.07) (xy 132.08 52.07)
 		)
@@
 	(wire
 		(pts
+			(xy 64.77 92.71) (xy 93.98 92.71)
+		)
+		(stroke
+			(width 0)
+			(type default)
+		)
+	)
+	(wire
+		(pts
+			(xy 93.98 85.09) (xy 99.06 85.09)
+		)
+		(stroke
+			(width 0)
+			(type default)
+		)
+	)
+	(wire
+		(pts
 			(xy 123.19 80.01) (xy 111.76 80.01)
-		)
-		(stroke
-			(width 0)
-			(type default)
-		)
-	)
-	(wire
-		(pts
-			(xy 115.57 92.71) (xy 115.57 85.09)
 		)
 		(stroke
@@
 		)
 	)
+	(hierarchical_label "PIT GATE"
+		(shape output)
+		(at 44.45 95.25 180)
+		(effects
+			(font
+				(size 1.27 1.27)
+			)
+			(justify right)
+		)
+	)
+	(hierarchical_label "PPI_O"
+		(shape input)
+		(at 49.53 34.29 180)
+		(effects
+			(font
+				(size 1.27 1.27)
+			)
+			(justify right)
+		)
+	)
 	(hierarchical_label "PIT OUT"
 		(shape input)
-		(at 44.45 95.25 180)
-		(effects
-			(font
-				(size 1.27 1.27)
-			)
-			(justify right)
-		)
-	)
-	(hierarchical_label "PPI_O[23:0]"
-		(shape input)
-		(at 49.53 34.29 180)
-		(effects
-			(font
-				(size 1.27 1.27)
-			)
-			(justify right)
-		)
-	)
-	(hierarchical_label "PIT GATE"
-		(shape input)
 		(at 44.45 92.71 180)
