File: rtc.kicad_sch (KiCad schematic)
At the start: 9 parts, among them IC1 DS12C887+, U2 74LS02, U37 74LS04, U47 74LS245, U50 74LS373

Commit message: Some house keeping
Connections:
- net GND: now also S2.4 (COM_2)
- net at IC1.21 (N.C._(~{RCLR)}), S2.1 (NO_1): now also S2.2 (NO_2)
- no-connect marks 9 -> 7
Changed lines of the file:
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@@
+	)
+	(junction
+		(at 215.9 71.12)
+		(diameter 0)
+		(color 0 0 0 0)
+	)
+	(junction
+		(at 214.63 77.47)
+		(diameter 0)
+		(color 0 0 0 0)
 	)
 	(junction
@@
 	)
 	(no_connect
-		(at 254 71.12)
-	)
-	(no_connect
 		(at 171.45 92.71)
 	)
@@
 	)
 	(no_connect
-		(at 254 73.66)
-	)
-	(no_connect
 		(at 201.93 95.25)
 	)
@@
 	(wire
 		(pts
+			(xy 264.16 71.12) (xy 254 71.12)
+		)
+		(stroke
+			(width 0)
+			(type default)
+		)
+	)
+	(wire
+		(pts
+			(xy 254 77.47) (xy 214.63 77.47)
+		)
+		(stroke
+			(width 0)
+			(type default)
+		)
+	)
+	(wire
+		(pts
 			(xy 158.75 59.69) (xy 154.94 59.69)
 		)
@@
 	(wire
 		(pts
+			(xy 264.16 59.69) (xy 264.16 71.12)
+		)
+		(stroke
+			(width 0)
+			(type default)
+		)
+	)
+	(wire
+		(pts
 			(xy 120.65 102.87) (xy 129.54 102.87)
 		)
@@
 	(wire
 		(pts
+			(xy 215.9 71.12) (xy 215.9 59.69)
+		)
+		(stroke
+			(width 0)
+			(type default)
+		)
+	)
+	(wire
+		(pts
 			(xy 124.46 54.61) (xy 129.54 54.61)
 		)
@@
 	(wire
 		(pts
-			(xy 212.09 71.12) (xy 223.52 71.12)
+			(xy 212.09 71.12) (xy 215.9 71.12)
 		)
 		(stroke
@@
 	(wire
 		(pts
+			(xy 254 73.66) (xy 254 77.47)
+		)
+		(stroke
+			(width 0)
+			(type default)
+		)
+	)
+	(wire
+		(pts
 			(xy 201.93 118.11) (xy 215.9 118.11)
 		)
@@
 	(wire
 		(pts
+			(xy 215.9 59.69) (xy 264.16 59.69)
+		)
+		(stroke
+			(width 0)
+			(type default)
+		)
+	)
+	(wire
+		(pts
 			(xy 154.94 52.07) (xy 160.02 52.07)
 		)
@@
 	(wire
 		(pts
-			(xy 214.63 97.79) (xy 214.63 73.66)
+			(xy 214.63 97.79) (xy 214.63 77.47)
 		)
 		(stroke
@@
 		)
 	)
+	(wire
+		(pts
+			(xy 214.63 77.47) (xy 214.63 73.66)
+		)
+		(stroke
+			(width 0)
+			(type default)
+		)
+	)
 	(bus
 		(pts
@@
 		)
 		(stroke
+			(width 0)
+			(type default)
+		)
+	)
+	(wire
+		(pts
+			(xy 215.9 71.12) (xy 223.52 71.12)
+		)
+		(stroke

Commit message: Upgraded speaker, esd protection, added dip sockets, adjusted routing
Parts:
- U2, U37: footprint Package_DIP:DIP-14_W7.62mm -> Package_DIP:DIP-14_W7.62mm_Socket
- U47, U50: footprint Package_DIP:DIP-20_W7.62mm -> Package_DIP:DIP-20_W7.62mm_Socket
Changed lines of the file:
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@@
 			)
 		)
-		(property "Footprint" "Package_DIP:DIP-14_W7.62mm"
+		(property "Footprint" "Package_DIP:DIP-14_W7.62mm_Socket"
 			(at 237.49 102.87 0)
 			(hide yes)
@@
 		)
 		(property "Sim.Type" ""
+			(at 237.49 102.87 0)
+			(hide yes)
+			(show_name no)
+			(do_not_autoplace no)
+			(effects
+				(font
+					(size 1.27 1.27)
+				)
+			)
+		)
+		(property "Sim.Device" ""
 			(at 237.49 102.87 0)
 			(hide yes)
@@
 			)
 		)
+		(property "Sim.Device" ""
+			(at 274.32 25.4 0)
+			(hide yes)
+			(show_name no)
+			(do_not_autoplace no)
+			(effects
+				(font
+					(size 1.27 1.27)
+				)
+			)
+		)
 		(pin "2"
 		)
@@
 			)
 		)
+		(property "Sim.Device" ""
+			(at 186.69 105.41 0)
+			(hide yes)
+			(show_name no)
+			(do_not_autoplace no)
+			(effects
+				(font
+					(size 1.27 1.27)
+				)
+			)
+		)
 		(pin "17"
 		)
@@
 			)
 		)
-		(property "Footprint" "Package_DIP:DIP-20_W7.62mm"
+		(property "Footprint" "Package_DIP:DIP-20_W7.62mm_Socket"
 			(at 142.24 107.95 0)
 			(hide yes)
@@
 		)
 		(property "Sim.Type" ""
+			(at 142.24 107.95 0)
+			(hide yes)
+			(show_name no)
+			(do_not_autoplace no)
+			(effects
+				(font
+					(size 1.27 1.27)
+				)
+			)
+		)
+		(property "Sim.Device" ""
 			(at 142.24 107.95 0)
 			(hide yes)
@@
 			)
 		)
+		(property "Sim.Device" ""
+			(at 260.35 25.4 0)
+			(hide yes)
+			(show_name no)
+			(do_not_autoplace no)
+			(effects
+				(font
+					(size 1.27 1.27)
+				)
+			)
+		)
 		(pin "2"
 		)
@@
 			)
 		)
-		(property "Footprint" "Package_DIP:DIP-20_W7.62mm"
+		(property "Footprint" "Package_DIP:DIP-20_W7.62mm_Socket"
 			(at 142.24 49.53 0)
 			(hide yes)
@@
 		)
 		(property "Sim.Type" ""
+			(at 142.24 49.53 0)
+			(hide yes)
+			(show_name no)
+			(do_not_autoplace no)
+			(effects
+				(font
+					(size 1.27 1.27)
+				)
+			)
+		)
+		(property "Sim.Device" ""
 			(at 142.24 49.53 0)
 			(hide yes)
@@
 			)
 		)
-		(property "Footprint" "Package_DIP:DIP-14_W7.62mm"
+		(property "Footprint" "Package_DIP:DIP-14_W7.62mm_Socket"
 			(at 76.2 77.47 0)
 			(hide yes)
@@
 		)
 		(property "Sim.Type" ""
+			(at 76.2 77.47 0)
+			(hide yes)
+			(show_name no)
+			(do_not_autoplace no)
+			(effects
+				(font
+					(size 1.27 1.27)
+				)
+			)
+		)
+		(property "Sim.Device" ""
 			(at 76.2 77.47 0)
 			(hide yes)
@@
 			)
 		)
+		(property "Sim.Device" ""
+			(at 223.52 71.12 0)
+			(hide yes)
+			(show_name no)
+			(do_not_autoplace no)
+			(effects
+				(font
+					(size 1.27 1.27)
+				)
+			)
+		)
 		(pin "1"
 		)
@@
 			)
 		)
-		(property "Footprint" "Package_DIP:DIP-14_W7.62mm"
+		(property "Footprint" "Package_DIP:DIP-14_W7.62mm_Socket"
 			(at 85.09 90.17 0)
 			(hide yes)
@@
 		)
 		(property "Sim.Type" ""
+			(at 85.09 90.17 0)
+			(hide yes)
+			(show_name no)
+			(do_not_autoplace no)
+			(effects
+				(font
+					(size 1.27 1.27)
+				)
+			)
+		)
+		(property "Sim.Device" ""
 			(at 85.09 90.17 0)
 			(hide yes)
@@
 			(at 246.38 25.4 0)
 			(hide yes)
+			(show_name no)
+			(do_not_autoplace no)
+			(effects
+				(font
+					(size 1.27 1.27)
+				)
+			)
+		)
+		(property "Sim.Device" ""
+			(at 246.38 25.4 0)
+			(hide yes)

Commit message: final commit before spinning
Changed lines of the file:
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@@
 	)
 	(hierarchical_label "RTC IRQ"
-		(shape input)
+		(shape output)
 		(at 254 102.87 0)
 		(effects
