File: isa_bus.kicad_sch (KiCad schematic)
At the start: 16 parts, among them J1 Bus_ISA_8bit, J2 Bus_ISA_8bit, J3 Bus_ISA_8bit, J4 Bus_ISA_8bit

Commit message: fixed things
Changed lines of the file:
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@@
 		)
 	)
+	(bus
+		(pts
+			(xy 162.56 67.31) (xy 162.56 72.39)
+		)
+		(stroke
+			(width 0)
+			(type default)
+		)
+	)
 	(wire
 		(pts
@@
 		)
 	)
-	(bus
-		(pts
-			(xy 162.56 64.77) (xy 162.56 72.39)
-		)
-		(stroke
-			(width 0)
-			(type default)
-		)
-	)
 	(wire
 		(pts
@@
 	)
 	(hierarchical_label "~{I{slash}O CH CK}"
-		(shape input)
+		(shape output)
 		(at 276.86 247.65 0)
 		(effects
@@
 	)
 	(hierarchical_label "I{slash}O CH RDY"
-		(shape input)
+		(shape output)
 		(at 278.13 52.07 0)
 		(effects
@@
 	)
 	(hierarchical_label "~{I{slash}O CH CK}"
-		(shape input)
+		(shape output)
 		(at 280.67 135.89 0)
 		(effects
@@
 	)
 	(hierarchical_label "IRQ[7..0]"
-		(shape input)
+		(shape output)
 		(at 146.05 191.77 180)
 		(effects
@@
 	)
 	(hierarchical_label "I{slash}O CH RDY"
-		(shape input)
+		(shape output)
 		(at 273.05 384.81 0)
 		(effects
@@
 	)
 	(hierarchical_label "~{I{slash}O CH CK}"
-		(shape input)
+		(shape output)
 		(at 273.05 359.41 0)
 		(effects
@@
 	)
 	(hierarchical_label "I{slash}O CH RDY"
-		(shape input)
+		(shape output)
 		(at 276.86 273.05 0)
 		(effects
@@
 	)
 	(hierarchical_label "IRQ[7..0]"
-		(shape input)
+		(shape output)
 		(at 138.43 415.29 180)
 		(effects
@@
 	)
 	(hierarchical_label "IRQ[7..0]"
-		(shape input)
+		(shape output)
 		(at 142.24 303.53 180)
 		(effects
@@
 	)
 	(hierarchical_label "I{slash}O CH RDY"
-		(shape input)
+		(shape output)
 		(at 280.67 161.29 0)
 		(effects
@@
 	)
 	(hierarchical_label "~{HRQ I{slash}O CH}"
-		(shape input)
+		(shape passive)
 		(at 143.51 46.99 180)
 		(effects
@@
 	)
 	(hierarchical_label "~{I{slash}O CH CK}"
-		(shape input)
+		(shape output)
 		(at 278.13 26.67 0)
 		(effects
@@
 	)
 	(hierarchical_label "~{HRQ I{slash}O CH}"
-		(shape input)
+		(shape passive)
 		(at 138.43 379.73 180)
 		(effects
@@
 	)
 	(hierarchical_label "~{HRQ I{slash}O CH}"
-		(shape input)
+		(shape passive)
 		(at 146.05 156.21 180)
 		(effects
@@
 	)
 	(hierarchical_label "~{HRQ I{slash}O CH}"
-		(shape input)
+		(shape passive)
 		(at 142.24 267.97 180)
 		(effects
@@
 	)
 	(hierarchical_label "IRQ[7..0]"
-		(shape input)
+		(shape output)
 		(at 143.51 82.55 180)
 		(effects

Commit message: final final review
Connections:
- net RESET DRV renamed RESET
Changed lines of the file:
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@@
 		)
 	)
-	(hierarchical_label "RESET DRV"
-		(shape input)
-		(at 147.32 140.97 180)
+	(hierarchical_label "RESET"
+		(shape input)
+		(at 144.78 31.75 180)
 		(effects
 			(font
@@
 		)
 	)
-	(hierarchical_label "RESET DRV"
-		(shape input)
-		(at 144.78 31.75 180)
-		(effects
-			(font
-				(size 1.27 1.27)
-			)
-			(justify right)
-		)
-	)
-	(hierarchical_label "RESET DRV"
+	(hierarchical_label "RESET"
 		(shape input)
 		(at 143.51 252.73 180)
@@
 		(shape output)
 		(at 146.05 191.77 180)
-		(effects
-			(font
-				(size 1.27 1.27)
-			)
-			(justify right)
-		)
-	)
-	(hierarchical_label "RESET DRV"
-		(shape input)
-		(at 139.7 364.49 180)
 		(effects
 			(font
@@
 		)
 	)
+	(hierarchical_label "RESET"
+		(shape input)
+		(at 147.32 140.97 180)
+		(effects
+			(font
+				(size 1.27 1.27)
+			)
+			(justify right)
+		)
+	)
 	(hierarchical_label "~{IOW}"
 		(shape input)
@@
 		)
 	)
+	(hierarchical_label "RESET"
+		(shape input)
+		(at 139.7 364.49 180)
+		(effects
+			(font
+				(size 1.27 1.27)
+			)
+			(justify right)
+		)
+	)
