File: processor_and_control.kicad_sch (KiCad schematic)
At the start: 38 parts, among them U13 8284, U14 8088_Max_Mode, U15 8087, U16 8259A, U18 74LS373, U19 74LS373, U20 74LS373, U21 74LS245, U23 8288, U24 74LS10, Y2 14.318 MHz

Commit message: fixed things
Connections:
- net ~{RDY WAIT} renamed ~{RDY}/WAIT
Other:
- moved on the sheet: R25, R26, R27, R28, R29, R43

Commit message: Upgraded speaker, esd protection, added dip sockets, adjusted routing
Parts:
- added R52: R, Resistor_SMD:R_1206_3216Metric_Pad1.30x1.75mm_HandSolder, symbol Device:R
- U13: footprint Package_DIP:DIP-18_W7.62mm -> Package_DIP:DIP-18_W7.62mm_Socket
- U14, U15: footprint Package_DIP:DIP-40_W15.24mm -> Package_DIP:DIP-40_W15.24mm_Socket
- U16: footprint Package_DIP:DIP-28_W15.24mm -> Package_DIP:DIP-28_W15.24mm_Socket
- U18, U19, U20, U21, U23: footprint Package_DIP:DIP-20_W7.62mm -> Package_DIP:DIP-20_W7.62mm_Socket
- U24: footprint Package_DIP:DIP-14_W7.62mm -> Package_DIP:DIP-14_W7.62mm_Socket
Connections:
- net ALE: now also R52.2; no longer U23.5 (ALE)
- new net: R52.1, U23.5 (ALE)
Other:
- note removed: "Decoupling Cap"
- moved on the sheet: C5

Commit message: final commit before spinning
Changed lines of the file:
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@@
 		)
 		(property "Footprint" "Package_DIP:DIP-40_W15.24mm_Socket"
-			(at 226.06 182.88 0)
+			(at 222.758 191.77 0)
+			(hide yes)
 			(show_name no)
 			(do_not_autoplace no)

Commit message: final final review
Parts:
- added C47, C48: 0.1 μF, Capacitor_SMD:C_1210_3225Metric_Pad1.33x2.70mm_HandSolder, symbol Device:C
- R44, R45, R46, R47, R48, R49, R50, R52: value R -> 33 Ω
Connections:
- net +5V: now also C47.1, C48.1
- net GND: now also C47.2, C48.2
- net RESET renamed RESET BRD
Other:
- moved on the sheet: R50
