File: retroslop.kicad_sch (KiCad schematic)
At the start: 9 parts

Commit message: tried manhattan routing
Connections:
- no-connect marks 1 -> 2
Other:
- sheet DMA ports: added ~{DACK[3..0]}; removed ~{DACK[3:0]}
- sheet ISA BUS ports: added ~{HRQ I/O CH}; removed none
Changed lines of the file:
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@@
 		(at 49.53 168.91)
 	)
+	(no_connect
+		(at 40.64 207.01)
+	)
 	(bus_entry
 		(at 208.28 283.21)
@@
 		)
 	)
+	(wire
+		(pts
+			(xy 40.64 207.01) (xy 52.07 207.01)
+		)
+		(stroke
+			(width 0)
+			(type default)
+		)
+	)
 	(bus
 		(pts
@@
 			)
 		)
+		(pin "~{HRQ I{slash}O CH}" input
+			(at 52.07 207.01 180)
+			(effects
+				(font
+					(size 1.27 1.27)
+				)
+				(justify left)
+			)
+		)
 		(instances
 			(project "retroslop"
@@
 			)
 		)
-		(pin "~{DACK[3:0]}" input
+		(pin "~{DACK[3..0]}" input
 			(at 168.91 153.67 180)
 			(effects

Commit message: finished routing rev3
Other:
- note added: "IO MAP 000-01F : DMA 020-03F : PIC 040-05F : PIT 060-07F : KBRD 080-09F : DMA REG 0A0-0BF : FLAG 0CF-0DF : PPI 0E0-0FF : UART 100-1FF : RTC"
Changed lines of the file:
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@@
 		)
 	)
+	(text "IO MAP\n000-01F : DMA\n020-03F : PIC\n040-05F : PIT\n060-07F : KBRD\n080-09F : DMA REG\n0A0-0BF : FLAG\n0CF-0DF : PPI\n0E0-0FF : UART\n100-1FF : RTC"
+		(exclude_from_sim no)
+		(at 240.538 91.694 0)
+		(effects
+			(font
+				(size 1.27 1.27)
+			)
+			(justify left)
+		)
+	)
 	(text "~{HRQ I/O CH} (or ~{NOWS})\nis unused in newer ibm variants"
 		(exclude_from_sim no)
@@
 		)
 	)
-	(label "~{CS4}"
+	(label "~{CS3}"
 		(at 199.39 148.59 0)
 		(effects
@@
 		)
 	)
-	(label "~{CS5}"
+	(label "~{CS4}"
 		(at 232.41 256.54 0)
 		(effects
@@
 			)
 		)
-		(pin "~{RTC CS}" input
+		(pin "~{RTC CS}" output
 			(at 195.58 101.6 0)
 			(effects
@@
 			)
 		)
-		(pin "~{DMA REG CS}" input
+		(pin "~{DMA REG CS}" output
 			(at 195.58 91.44 0)
 			(effects
@@
 			)
 		)
-		(pin "~{PPI CS}" input
+		(pin "~{PPI CS}" output
 			(at 195.58 96.52 0)
 			(effects
@@
 			)
 		)
-		(pin "~{PIT CS}" input
+		(pin "~{PIT CS}" output
 			(at 195.58 86.36 0)
 			(effects
@@
 			)
 		)
-		(pin "~{KBRD CS}" input
+		(pin "~{KBRD CS}" output
 			(at 195.58 88.9 0)
 			(effects
@@
 			)
 		)
-		(pin "~{DMA CS}" input
+		(pin "~{DMA CS}" output
 			(at 195.58 83.82 0)
 			(effects
@@
 			)
 		)
-		(pin "~{FLAG CS}" input
+		(pin "~{FLAG CS}" output
 			(at 195.58 93.98 0)
 			(effects
@@
 			)
 		)
-		(pin "~{UART CS}" input
+		(pin "~{UART CS}" output
 			(at 195.58 99.06 0)
 			(effects

Commit message: Some house keeping
Changed lines of the file:
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@@
-		)
-	)
-	(label "~{XIOR}"
-		(at 237.49 283.21 180)
-		(effects
-			(font
-				(size 1.27 1.27)
-			)
-			(justify right bottom)
 		)
 	)
@@
 	(label "~{XIOW}"
 		(at 237.49 320.04 180)
+		(effects
+			(font
+				(size 1.27 1.27)
+			)
+			(justify right bottom)
+		)
+	)
+	(label "~{XIOW}"
+		(at 237.49 283.21 180)
 		(effects
 			(font
@@
 		)
 	)
-	(label "~{XIOW}"
-		(at 237.49 285.75 180)
-		(effects
-			(font
-				(size 1.27 1.27)
-			)
-			(justify right bottom)
-		)
-	)
 	(label "~{XMEMR}"
 		(at 92.71 153.67 0)
@@
 		)
 	)
+	(label "~{XIOR}"
+		(at 237.49 285.75 180)
+		(effects
+			(font
+				(size 1.27 1.27)
+			)
+			(justify right bottom)
+		)
+	)

Commit message: fixed things
Other:
- sheet Processor And Control ports: added ~{RDY}/WAIT; removed ~{RDY WAIT}

Commit message: Upgraded speaker, esd protection, added dip sockets, adjusted routing
Changed lines of the file:
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@@
 	)
 	(junction
+		(at 128.27 162.56)
+		(diameter 0)
+		(color 0 0 0 0)
+	)
+	(junction
 		(at 219.71 309.88)
 		(diameter 0)
@@
 	)
 	(junction
-		(at 128.27 163.83)
-		(diameter 0)
-		(color 0 0 0 0)
-	)
-	(junction
 		(at 135.89 57.15)
 		(diameter 0)
@@
 	(bus
 		(pts
-			(xy 128.27 163.83) (xy 100.33 163.83)
+			(xy 128.27 162.56) (xy 100.33 162.56)
 		)
 		(stroke
@@
 	(bus
 		(pts
-			(xy 100.33 156.21) (xy 100.33 163.83)
+			(xy 100.33 156.21) (xy 100.33 162.56)
 		)
 		(stroke
@@
 	(bus
 		(pts
+			(xy 128.27 162.56) (xy 128.27 228.6)
+		)
+		(stroke
+			(width 0)
+			(type default)
+		)
+	)
+	(bus
+		(pts
 			(xy 217.17 280.67) (xy 229.87 280.67)
 		)
@@
 		)
 	)
-	(bus
-		(pts
-			(xy 128.27 163.83) (xy 128.27 228.6)
-		)
-		(stroke
-			(width 0)
-			(type default)
-		)
-	)
 	(wire
 		(pts
@@
 	(bus
 		(pts
-			(xy 128.27 100.33) (xy 128.27 163.83)
+			(xy 128.27 100.33) (xy 128.27 162.56)
 		)
 		(stroke
@@
 			)
 		)
+		(property "Sim.Device" ""
+			(at 21.59 398.78 0)
+			(hide yes)
+			(show_name no)
+			(do_not_autoplace no)
+			(effects
+				(font
+					(size 1.27 1.27)
+				)
+			)
+		)
 		(instances
 			(project "retroslop"
@@
 			)
 		)
+		(property "Sim.Device" ""
+			(at 21.59 378.46 0)
+			(hide yes)
+			(show_name no)
+			(do_not_autoplace no)
+			(effects
+				(font
+					(size 1.27 1.27)
+				)
+			)
+		)
 		(instances
 			(project "retroslop"
@@
 			)
 		)
+		(property "Sim.Device" ""
+			(at 21.59 388.62 0)
+			(hide yes)
+			(show_name no)
+			(do_not_autoplace no)
+			(effects
+				(font
+					(size 1.27 1.27)
+				)
+			)
+		)
 		(instances
 			(project "retroslop"
@@
 			)
 		)
+		(property "Sim.Device" ""
+			(at 21.59 393.7 0)
+			(hide yes)
+			(show_name no)
+			(do_not_autoplace no)
+			(effects
+				(font
+					(size 1.27 1.27)
+				)
+			)
+		)
 		(instances
 			(project "retroslop"
@@
 			)
 		)
+		(property "Sim.Device" ""
+			(at 21.59 358.14 0)
+			(hide yes)
+			(show_name no)
+			(do_not_autoplace no)
+			(effects
+				(font
+					(size 1.27 1.27)
+				)
+			)
+		)
 		(instances
 			(project "retroslop"
@@
 			)
 		)
+		(property "Sim.Device" ""
+			(at 21.59 383.54 0)
+			(hide yes)
+			(show_name no)
+			(do_not_autoplace no)
+			(effects
+				(font
+					(size 1.27 1.27)
+				)
+			)
+		)
 		(instances
 			(project "retroslop"
@@
 			)
 		)
+		(property "Sim.Device" ""
+			(at 21.59 363.22 0)
+			(hide yes)
+			(show_name no)
+			(do_not_autoplace no)
+			(effects
+				(font
+					(size 1.27 1.27)
+				)
+			)
+		)
 		(instances
 			(project "retroslop"
@@
 			)
 		)
+		(property "Sim.Device" ""
+			(at 21.59 373.38 0)
+			(hide yes)
+			(show_name no)
+			(do_not_autoplace no)
+			(effects
+				(font
+					(size 1.27 1.27)
+				)
+			)
+		)
 		(instances
 			(project "retroslop"
@@
 			(at 21.59 368.3 0)
 			(hide yes)
+			(show_name no)
+			(do_not_autoplace no)
+			(effects
+				(font
+					(size 1.27 1.27)
+				)
+			)
+		)
+		(property "Sim.Device" ""
+			(at 21.59 368.3 0)
+			(hide yes)

Commit message: final commit before spinning
Other:
- sheet Pinout ports: added PPI_O; removed PPI_O[23:0]
- sheet Programmable Peripheral Interface ports: added PPI_O, XA[9..0]; removed PPI_O[23..0], XA[19..0]
Changed lines of the file:
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@@
 	(text "IO MAP\n000-01F : DMA\n020-03F : PIC\n040-05F : PIT\n060-07F : KBRD\n080-09F : DMA REG\n0A0-0BF : FLAG\n0CF-0DF : PPI\n0E0-0FF : UART\n100-1FF : RTC"
 		(exclude_from_sim no)
-		(at 240.538 91.694 0)
+		(at 248.158 125.476 0)
 		(effects
 			(font
@@
 	(wire
 		(pts
-			(xy 266.7 349.25) (xy 274.32 349.25)
-		)
-		(stroke
-			(width 0)
-			(type default)
-		)
-	)
-	(wire
-		(pts
 			(xy 102.87 102.87) (xy 102.87 165.1)
 		)
@@
 	(bus
 		(pts
+			(xy 266.7 349.25) (xy 274.32 349.25)
+		)
+		(stroke
+			(width 0)
+			(type default)
+		)
+	)
+	(bus
+		(pts
 			(xy 208.28 241.3) (xy 217.17 241.3)
 		)
@@
 		)
 	)
-	(wire
+	(bus
 		(pts
-			(xy 232.41 294.64) (xy 240.03 294.64)
+			(xy 274.32 349.25) (xy 274.32 279.4)
 		)
 		(stroke
@@
 	(wire
 		(pts
-			(xy 93.98 213.36) (xy 90.17 213.36)
+			(xy 232.41 294.64) (xy 240.03 294.64)
 		)
 		(stroke
@@
 	(wire
 		(pts
-			(xy 212.09 289.56) (xy 212.09 332.74)
+			(xy 93.98 213.36) (xy 90.17 213.36)
 		)
 		(stroke
@@
 	(wire
 		(pts
-			(xy 92.71 123.19) (xy 147.32 123.19)
+			(xy 212.09 289.56) (xy 212.09 332.74)
 		)
 		(stroke
@@
 	(wire
 		(pts
-			(xy 274.32 349.25) (xy 274.32 279.4)
+			(xy 92.71 123.19) (xy 147.32 123.19)
 		)
 		(stroke
@@
 		)
 	)
-	(wire
-		(pts
-			(xy 274.32 279.4) (xy 266.7 279.4)
-		)
-		(stroke
-			(width 0)
-			(type default)
-		)
-	)
 	(bus
 		(pts
@@
 	(bus
 		(pts
+			(xy 274.32 279.4) (xy 266.7 279.4)
+		)
+		(stroke
+			(width 0)
+			(type default)
+		)
+	)
+	(bus
+		(pts
 			(xy 135.89 115.57) (xy 135.89 167.64)
 		)
@@
 			)
 		)
-		(pin "PIT OUT" input
+		(pin "PIT OUT" output
 			(at 266.7 326.39 0)
 			(effects
@@
 			)
 		)
-		(pin "PPI_O[23..0]" input
+		(pin "PPI_O" bidirectional
 			(at 266.7 279.4 0)
 			(effects
@@
 			)
 		)
-		(pin "XA[19..0]" input
+		(pin "XA[9..0]" input
 			(at 240.03 274.32 180)
 			(effects
@@
 			)
 		)
-		(pin "XA[9..0]" input
+		(pin "XA[9..0]" tri_state
 			(at 195.58 72.39 0)
 			(effects
@@
 			)
 		)
-		(pin "XD[7..0]" input
+		(pin "XD[7..0]" tri_state
 			(at 195.58 118.11 0)
 			(effects
@@
 			)
 		)
-		(pin "XA[9..0]" input
+		(pin "XA[9..0]" tri_state
 			(at 195.58 115.57 0)
 			(effects
@@
 			)
 		)
-		(pin "ENABLE IO CK" input
+		(pin "ENABLE IO CK" output
 			(at 266.7 241.3 0)
 			(effects
@@
 			)
 		)
-		(pin "ALLOW NMI" input
+		(pin "ALLOW NMI" output
 			(at 266.7 236.22 0)
 			(effects
@@
 			)
 		)
-		(pin "PPI_O[23:0]" input
+		(pin "PPI_O" input
 			(at 266.7 349.25 0)
 			(effects
@@
 			)
 		)
-		(pin "PIT GATE" input
+		(pin "PIT GATE" output
 			(at 266.7 344.17 0)
 			(effects
@@
 			)
 		)
-		(pin "RTC IRQ" input
+		(pin "RTC IRQ" output
 			(at 195.58 290.83 0)
 			(effects

Commit message: final final review
Other:
- sheet ISA BUS ports: added RESET; removed RESET DRV
- sheet Processor And Control ports: added RESET BRD; removed RESET
- sheet Wait State Generator ports: added RESET BRD; removed RESET
- moved on the sheet: H1, H2, H3, H4, H5, H6, H7, H8, H9
