File: ros_and_bus_driver.kicad_sch (KiCad schematic)
At the start: 14 parts, among them U17 74LS32, U27 74LS245, U28 74LS245, U48 74LS244, U56 74LS244

Commit message: fixed things
Other:
- note added: "When an IO read happens we need to read from XD but when XA9 is asserted that's a read from the isa bus so we don't want double drivers"
- note removed: "(IOR & ~XA9) | (RAS & MEMR) = DIR IOR & ~XA9 = DIR ~(~IOR | XA9) = DIR IOR & ~XA9 = ~TOA ~(IOR & ~XA9) If (IOR == 0 and XA9 == 0) { A->B = 0 } ~(A->B) = ~IOR & ~XA9 A->B = ~(~IOR & ~XA9) IOR | XA9 = A->B"
Changed lines of the file:
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@@
 	(generator_version "10.0")
 	(paper "A4" portrait)
-	(text "(IOR & ~XA9) | (RAS & MEMR) = DIR\nIOR & ~XA9 = DIR\n~(~IOR | XA9) = DIR\nIOR & ~XA9 = ~TOA\n~(IOR & ~XA9)\n\nIf (IOR == 0 and XA9 == 0) {\n	A->B = 0\n}\n\n~(A->B) = ~IOR & ~XA9\n\nA->B = ~(~IOR & ~XA9)\nIOR | XA9 = A->B"
+	(text "When an IO read happens we need to read from XD\nbut when XA9 is asserted that's a read from the \nisa bus so we don't want double drivers"
 		(exclude_from_sim no)
-		(at 158.242 76.454 0)
+		(at 150.622 58.928 0)
 		(effects
 			(font
 				(size 1.27 1.27)
 			)
-			(justify left)
 		)
 	)
@@
 		(color 0 0 0 0)
 	)
+	(junction
+		(at 66.04 180.34)
+		(diameter 0)
+		(color 0 0 0 0)
+	)
 	(no_connect
 		(at 104.14 52.07)
@@
 	(wire
 		(pts
-			(xy 118.11 76.2) (xy 130.81 76.2)
+			(xy 118.11 76.2) (xy 140.97 76.2)
 		)
 		(stroke
@@
 	(wire
 		(pts
-			(xy 152.4 85.09) (xy 66.04 85.09)
+			(xy 166.37 85.09) (xy 66.04 85.09)
 		)
 		(stroke
@@
 	(wire
 		(pts
-			(xy 118.11 71.12) (xy 130.81 71.12)
+			(xy 118.11 71.12) (xy 140.97 71.12)
 		)
 		(stroke
@@
 	(wire
 		(pts
+			(xy 66.04 180.34) (xy 66.04 217.17)
+		)
+		(stroke
+			(width 0)
+			(type default)
+		)
+	)
+	(wire
+		(pts
 			(xy 66.04 177.8) (xy 66.04 180.34)
 		)
@@
 	(wire
 		(pts
-			(xy 50.8 44.45) (xy 78.74 44.45)
+			(xy 66.04 217.17) (xy 78.74 217.17)
 		)
 		(stroke
@@
 		)
 	)
-	(bus
+	(wire
 		(pts
-			(xy 69.85 152.4) (xy 69.85 209.55)
+			(xy 50.8 44.45) (xy 78.74 44.45)
 		)
 		(stroke
@@
 		)
 	)
-	(wire
+	(bus
 		(pts
-			(xy 91.44 77.47) (xy 91.44 76.2)
+			(xy 69.85 152.4) (xy 69.85 209.55)
 		)
 		(stroke
@@
 	(wire
 		(pts
-			(xy 146.05 73.66) (xy 152.4 73.66)
+			(xy 91.44 77.47) (xy 91.44 76.2)
 		)
 		(stroke
@@
 	(wire
 		(pts
-			(xy 110.49 170.18) (xy 104.14 170.18)
+			(xy 156.21 73.66) (xy 166.37 73.66)
 		)
 		(stroke
@@
 	(wire
 		(pts
-			(xy 50.8 125.73) (xy 66.04 125.73)
+			(xy 110.49 170.18) (xy 104.14 170.18)
 		)
 		(stroke
@@
 	(wire
 		(pts
-			(xy 50.8 217.17) (xy 78.74 217.17)
+			(xy 50.8 125.73) (xy 66.04 125.73)
 		)
 		(stroke
@@
 	(wire
 		(pts
-			(xy 152.4 73.66) (xy 152.4 85.09)
+			(xy 166.37 73.66) (xy 166.37 85.09)
 		)
 		(stroke
@@
 		)
 	)
-	(hierarchical_label "AEN BRD"
-		(shape input)
-		(at 50.8 217.17 180)
-		(effects
-			(font
-				(size 1.27 1.27)
-			)
-			(justify right)
-		)
-	)
 	(hierarchical_label "~{IOW}"
 		(shape input)
@@
 	(symbol
 		(lib_id "74xx:74LS32")
-		(at 138.43 73.66 0)
+		(at 148.59 73.66 0)
 		(unit 1)
-		(body_style 1)
+		(body_style 2)
 		(exclude_from_sim no)
 		(in_bom yes)
@@
 		(fields_autoplaced yes)
 		(property "Reference" "U17"
-			(at 138.43 64.77 0)
+			(at 148.59 64.77 0)
 			(show_name no)
 			(do_not_autoplace no)
@@
 		)
 		(property "Value" "74LS32"
-			(at 138.43 67.31 0)
+			(at 148.59 67.31 0)
 			(show_name no)
 			(do_not_autoplace no)
@@
 		)
 		(property "Footprint" "Package_DIP:DIP-14_W7.62mm"
-			(at 138.43 73.66 0)
+			(at 148.59 73.66 0)
 			(hide yes)
 			(show_name no)
@@
 		)
 		(property "Datasheet" "http://www.ti.com/lit/gpn/sn74LS32"
-			(at 138.43 73.66 0)
+			(at 148.59 73.66 0)
 			(hide yes)
 			(show_name no)
@@
 		)
 		(property "Description" "Quad 2-input OR"
-			(at 138.43 73.66 0)
+			(at 148.59 73.66 0)
 			(hide yes)
 			(show_name no)

Commit message: Upgraded speaker, esd protection, added dip sockets, adjusted routing
Parts:
- U17: footprint Package_DIP:DIP-14_W7.62mm -> Package_DIP:DIP-14_W7.62mm_Socket
- U27, U28, U48, U56: footprint Package_DIP:DIP-20_W7.62mm -> Package_DIP:DIP-20_W7.62mm_Socket
Changed lines of the file:
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@@
+			)
+		)
+		(property "Sim.Device" ""
+			(at 120.65 34.29 0)
+			(hide yes)
+			(show_name no)
+			(do_not_autoplace no)
+			(effects
+				(font
+					(size 1.27 1.27)
+				)
 			)
 		)
@@
 			)
 		)
+		(property "Sim.Device" ""
+			(at 17.78 273.05 0)
+			(hide yes)
+			(show_name no)
+			(do_not_autoplace no)
+			(effects
+				(font
+					(size 1.27 1.27)
+				)
+			)
+		)
 		(pin "2"
 		)
@@
 			)
 		)
+		(property "Sim.Device" ""
+			(at 127 214.63 90)
+			(hide yes)
+			(show_name no)
+			(do_not_autoplace no)
+			(effects
+				(font
+					(size 1.27 1.27)
+				)
+			)
+		)
 		(pin "1"
 		)
@@
 			)
 		)
+		(property "Sim.Device" ""
+			(at 31.75 273.05 0)
+			(hide yes)
+			(show_name no)
+			(do_not_autoplace no)
+			(effects
+				(font
+					(size 1.27 1.27)
+				)
+			)
+		)
 		(pin "2"
 		)
@@
 			)
 		)
+		(property "Sim.Device" ""
+			(at 154.94 34.29 0)
+			(hide yes)
+			(show_name no)
+			(do_not_autoplace no)
+			(effects
+				(font
+					(size 1.27 1.27)
+				)
+			)
+		)
 		(pin "1"
 		)
@@
 			)
 		)
-		(property "Footprint" "Package_DIP:DIP-20_W7.62mm"
+		(property "Footprint" "Package_DIP:DIP-20_W7.62mm_Socket"
 			(at 91.44 222.25 0)
 			(hide yes)
@@
 			)
 		)
+		(property "Sim.Device" ""
+			(at 91.44 222.25 0)
+			(hide yes)
+			(show_name no)
+			(do_not_autoplace no)
+			(effects
+				(font
+					(size 1.27 1.27)
+				)
+			)
+		)
 		(pin "19"
 		)
@@
 			)
 		)
-		(property "Footprint" "Package_DIP:DIP-20_W7.62mm"
+		(property "Footprint" "Package_DIP:DIP-20_W7.62mm_Socket"
 			(at 91.44 54.61 0)
 			(hide yes)
@@
 			)
 		)
+		(property "Sim.Device" ""
+			(at 91.44 54.61 0)
+			(hide yes)
+			(show_name no)
+			(do_not_autoplace no)
+			(effects
+				(font
+					(size 1.27 1.27)
+				)
+			)
+		)
 		(pin "5"
 		)
@@
 			)
 		)
-		(property "Footprint" "Package_DIP:DIP-20_W7.62mm"
+		(property "Footprint" "Package_DIP:DIP-20_W7.62mm_Socket"
 			(at 91.44 167.64 0)
 			(hide yes)
@@
 			)
 		)
+		(property "Sim.Device" ""
+			(at 91.44 167.64 0)
+			(hide yes)
+			(show_name no)
+			(do_not_autoplace no)
+			(effects
+				(font
+					(size 1.27 1.27)
+				)
+			)
+		)
 		(pin "19"
 		)
@@
 			)
 		)
+		(property "Sim.Device" ""
+			(at 132.08 34.29 0)
+			(hide yes)
+			(show_name no)
+			(do_not_autoplace no)
+			(effects
+				(font
+					(size 1.27 1.27)
+				)
+			)
+		)
 		(pin "1"
 		)
@@
 			)
 		)
+		(property "Sim.Device" ""
+			(at 143.51 34.29 0)
+			(hide yes)
+			(show_name no)
+			(do_not_autoplace no)
+			(effects
+				(font
+					(size 1.27 1.27)
+				)
+			)
+		)
 		(pin "1"
 		)
@@
 			)
 		)
+		(property "Sim.Device" ""
+			(at 45.72 273.05 0)
+			(hide yes)
+			(show_name no)
+			(do_not_autoplace no)
+			(effects
+				(font
+					(size 1.27 1.27)
+				)
+			)
+		)
 		(pin "2"
 		)
@@
 			)
 		)
-		(property "Footprint" "Package_DIP:DIP-20_W7.62mm"
+		(property "Footprint" "Package_DIP:DIP-20_W7.62mm_Socket"
 			(at 91.44 113.03 0)
 			(hide yes)
@@
 			)
 		)
+		(property "Sim.Device" ""
+			(at 91.44 113.03 0)
+			(hide yes)
+			(show_name no)
+			(do_not_autoplace no)
+			(effects
+				(font
+					(size 1.27 1.27)
+				)
+			)
+		)
 		(pin "5"
 		)
@@
 			)
 		)
-		(property "Footprint" "Package_DIP:DIP-14_W7.62mm"
+		(property "Footprint" "Package_DIP:DIP-14_W7.62mm_Socket"
 			(at 148.59 73.66 0)
 			(hide yes)
@@
 			)
 		)
+		(property "Sim.Device" ""
+			(at 148.59 73.66 0)
+			(hide yes)
+			(show_name no)
+			(do_not_autoplace no)
+			(effects
+				(font
+					(size 1.27 1.27)
+				)
+			)
+		)
 		(pin "7"
 		)
@@
 			(at 59.69 273.05 0)
 			(hide yes)
+			(show_name no)
+			(do_not_autoplace no)
+			(effects
+				(font
+					(size 1.27 1.27)
+				)
+			)
+		)
+		(property "Sim.Device" ""
+			(at 59.69 273.05 0)
+			(hide yes)

Commit message: final final review
Parts:
- R51: value R -> 33 Ω
Other:
- moved on the sheet: C63, C64, C65, C66, R37, R38, R39, R40, R51, U17A, U27, U28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
