File: uart.kicad_sch (KiCad schematic)
At the start: 9 parts, among them J5 DE9_Socket, U42 16550, U43 MAX232

Commit message: Upgraded speaker, esd protection, added dip sockets, adjusted routing
Parts:
- U42: footprint Package_DIP:DIP-40_W15.24mm -> Package_DIP:DIP-40_W15.24mm_Socket
- U43: footprint Package_DIP:DIP-16_W7.62mm -> Package_DIP:DIP-16_W7.62mm_Socket
Changed lines of the file:
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@@
+			)
+		)
+		(property "Sim.Device" ""
+			(at 256.54 29.21 0)
+			(hide yes)
+			(show_name no)
+			(do_not_autoplace no)
+			(effects
+				(font
+					(size 1.27 1.27)
+				)
 			)
 		)
@@
 			)
 		)
-		(property "Footprint" "Package_DIP:DIP-40_W15.24mm"
+		(property "Footprint" "Package_DIP:DIP-40_W15.24mm_Socket"
 			(at 102.87 105.41 0)
 			(hide yes)
@@
 		)
 		(property "Sim.Type" ""
+			(at 102.87 105.41 0)
+			(hide yes)
+			(show_name no)
+			(do_not_autoplace no)
+			(effects
+				(font
+					(size 1.27 1.27)
+				)
+			)
+		)
+		(property "Sim.Device" ""
 			(at 102.87 105.41 0)
 			(hide yes)
@@
 			)
 		)
-		(property "Footprint" "Package_DIP:DIP-16_W7.62mm"
+		(property "Footprint" "Package_DIP:DIP-16_W7.62mm_Socket"
 			(at 181.61 114.3 0)
 			(hide yes)
@@
 		)
 		(property "Sim.Type" ""
+			(at 180.34 87.63 0)
+			(hide yes)
+			(show_name no)
+			(do_not_autoplace no)
+			(effects
+				(font
+					(size 1.27 1.27)
+				)
+			)
+		)
+		(property "Sim.Device" ""
 			(at 180.34 87.63 0)
 			(hide yes)
@@
 			)
 		)
+		(property "Sim.Device" ""
+			(at 247.65 95.25 0)
+			(hide yes)
+			(show_name no)
+			(do_not_autoplace no)
+			(effects
+				(font
+					(size 1.27 1.27)
+				)
+			)
+		)
 		(pin "8"
 		)
@@
 			)
 		)
+		(property "Sim.Device" ""
+			(at 153.67 68.58 0)
+			(hide yes)
+			(show_name no)
+			(do_not_autoplace no)
+			(effects
+				(font
+					(size 1.27 1.27)
+				)
+			)
+		)
 		(pin "2"
 		)
@@
 			)
 		)
+		(property "Sim.Device" ""
+			(at 219.71 114.3 0)
+			(hide yes)
+			(show_name no)
+			(do_not_autoplace no)
+			(effects
+				(font
+					(size 1.27 1.27)
+				)
+			)
+		)
 		(pin "2"
 		)
@@
 			)
 		)
+		(property "Sim.Device" ""
+			(at 205.74 68.58 0)
+			(hide yes)
+			(show_name no)
+			(do_not_autoplace no)
+			(effects
+				(font
+					(size 1.27 1.27)
+				)
+			)
+		)
 		(pin "2"
 		)
@@
 			)
 		)
+		(property "Sim.Device" ""
+			(at 270.51 29.21 0)
+			(hide yes)
+			(show_name no)
+			(do_not_autoplace no)
+			(effects
+				(font
+					(size 1.27 1.27)
+				)
+			)
+		)
 		(pin "2"
 		)
@@
 			(at 207.01 114.3 0)
 			(hide yes)
+			(show_name no)
+			(do_not_autoplace no)
+			(effects
+				(font
+					(size 1.27 1.27)
+				)
+			)
+		)
+		(property "Sim.Device" ""
+			(at 207.01 114.3 0)
+			(hide yes)

Commit message: final final review
Other:
- moved on the sheet: C52
Changed lines of the file:
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@@
 	(wire
 		(pts
-			(xy 153.67 72.39) (xy 160.02 72.39)
+			(xy 151.13 72.39) (xy 160.02 72.39)
 		)
 		(stroke
@@
 	(wire
 		(pts
-			(xy 153.67 64.77) (xy 160.02 64.77)
+			(xy 151.13 64.77) (xy 160.02 64.77)
 		)
 		(stroke
@@
 	(symbol
 		(lib_id "Device:C")
-		(at 153.67 68.58 0)
+		(at 151.13 68.58 0)
 		(unit 1)
 		(body_style 1)
@@
 		(fields_autoplaced yes)
 		(property "Reference" "C52"
-			(at 157.48 67.3099 0)
+			(at 154.94 67.3099 0)
 			(show_name no)
 			(do_not_autoplace no)
@@
 		)
 		(property "Value" "1 μF"
-			(at 157.48 69.8499 0)
+			(at 154.94 69.8499 0)
 			(show_name no)
 			(do_not_autoplace no)
@@
 		)
 		(property "Footprint" "Capacitor_SMD:C_1210_3225Metric_Pad1.33x2.70mm_HandSolder"
-			(at 154.6352 72.39 0)
+			(at 152.0952 72.39 0)
 			(hide yes)
 			(show_name no)
@@
 		)
 		(property "Datasheet" ""
-			(at 153.67 68.58 0)
+			(at 151.13 68.58 0)
 			(hide yes)
 			(show_name no)
@@
 		)
 		(property "Description" "Unpolarized capacitor"
-			(at 153.67 68.58 0)
+			(at 151.13 68.58 0)
 			(hide yes)
 			(show_name no)
@@
 		)
 		(property "Sim.Type" ""
-			(at 153.67 68.58 0)
+			(at 151.13 68.58 0)
 			(hide yes)
 			(show_name no)
@@
 		)
 		(property "Sim.Device" ""
-			(at 153.67 68.58 0)
-			(hide yes)
-			(show_name no)
+			(at 151.13 68.58 0)
+			(hide yes)
+			(show_name no)
