File: wait_state_generator.kicad_sch (KiCad schematic)
At the start: 23 parts, among them J12 FPU JUMPER, U1 74LS00, U10 74LS74, U2 74LS02, U22 74LS04, U29 74LS20, U3 74LS30, U32 74LS175, U37 74LS04, U4 74LS00

Commit message: Progress routing
Connections:
- net +5V: no longer J12.1 (Pin_1), U1.5
- new net FPU INSTL: J12.1 (Pin_1), U1.5
Changed lines of the file:
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@@
 	)
 	(junction
-		(at 118.11 137.16)
-		(diameter 0)
-		(color 0 0 0 0)
-	)
-	(junction
-		(at 121.92 153.67)
-		(diameter 0)
-		(color 0 0 0 0)
-	)
-	(junction
 		(at 113.03 226.06)
 		(diameter 0)
@@
 	)
 	(junction
-		(at 52.07 250.19)
-		(diameter 0)
-		(color 0 0 0 0)
-	)
-	(junction
 		(at 55.88 179.07)
 		(diameter 0)
@@
 	(wire
 		(pts
-			(xy 118.11 137.16) (xy 118.11 176.53)
-		)
-		(stroke
-			(width 0)
-			(type default)
-		)
-	)
-	(wire
-		(pts
 			(xy 311.15 181.61) (xy 311.15 185.42)
 		)
@@
 	(wire
 		(pts
-			(xy 121.92 171.45) (xy 147.32 171.45)
-		)
-		(stroke
-			(width 0)
-			(type default)
-		)
-	)
-	(wire
-		(pts
 			(xy 204.47 129.54) (xy 226.06 129.54)
 		)
@@
 	(wire
 		(pts
-			(xy 52.07 250.19) (xy 39.37 250.19)
-		)
-		(stroke
-			(width 0)
-			(type default)
-		)
-	)
-	(wire
-		(pts
 			(xy 38.1 132.08) (xy 77.47 132.08)
 		)
@@
 	(wire
 		(pts
-			(xy 52.07 250.19) (xy 82.55 250.19)
+			(xy 39.37 250.19) (xy 82.55 250.19)
 		)
 		(stroke
@@
 	(wire
 		(pts
-			(xy 52.07 247.65) (xy 52.07 250.19)
-		)
-		(stroke
-			(width 0)
-			(type default)
-		)
-	)
-	(wire
-		(pts
 			(xy 38.1 184.15) (xy 68.58 184.15)
 		)
@@
 	(wire
 		(pts
-			(xy 118.11 176.53) (xy 147.32 176.53)
-		)
-		(stroke
-			(width 0)
-			(type default)
-		)
-	)
-	(wire
-		(pts
 			(xy 214.63 97.79) (xy 166.37 97.79)
 		)
@@
 		)
 	)
-	(wire
-		(pts
-			(xy 121.92 153.67) (xy 121.92 171.45)
-		)
-		(stroke
-			(width 0)
-			(type default)
-		)
-	)
 	(label "~{CLK}"
 		(at 247.65 153.67 0)
@@
 		)
 	)
-	(label "CLK"
-		(at 142.24 176.53 0)
-		(effects
-			(font
-				(size 1.27 1.27)
-			)
-			(justify left bottom)
-		)
-	)
 	(label "AEN"
 		(at 207.01 116.84 0)
@@
 		)
 	)
-	(label "~{CLK}"
-		(at 142.24 171.45 0)
-		(effects
-			(font
-				(size 1.27 1.27)
-			)
-			(justify left bottom)
-		)
-	)
 	(label "HOLDA"
 		(at 172.72 116.84 0)
@@
 		(at 260.35 68.58 0)
 		(unit 4)
-		(body_style 1)
+		(body_style 2)
 		(exclude_from_sim no)
 		(in_bom yes)
@@
 				)
 			)
-		)
-	)
-	(symbol
-		(lib_id "power:VCC")
-		(at 52.07 247.65 0)
-		(unit 1)
-		(body_style 1)
-		(exclude_from_sim no)
-		(in_bom yes)
-		(on_board yes)
-		(in_pos_files yes)
-		(dnp no)
-		(fields_autoplaced yes)
-		(property "Reference" "#PWR0101"
-			(at 52.07 251.46 0)
-			(hide yes)
-			(show_name no)
-			(do_not_autoplace no)
-			(effects
-				(font
-					(size 1.27 1.27)
-				)
-			)
-		)
-		(property "Value" "+5V"
-			(at 52.07 242.57 0)
-			(show_name no)
-			(do_not_autoplace no)
-			(effects
-				(font
-					(size 1.27 1.27)
-				)
-			)
-		)
-		(property "Footprint" ""
-			(at 52.07 247.65 0)
-			(hide yes)
-			(show_name no)
-			(do_not_autoplace no)
-			(effects
-				(font
-					(size 1.27 1.27)
-				)
-			)
-		)
-		(property "Datasheet" ""
-			(at 52.07 247.65 0)
-			(hide yes)
-			(show_name no)
-			(do_not_autoplace no)
-			(effects
-				(font
-					(size 1.27 1.27)
-				)
-			)
-		)
-		(property "Description" "Power symbol creates a global label with name \"VCC\""
-			(at 52.07 247.65 0)
-			(hide yes)
-			(show_name no)
-			(do_not_autoplace no)
-			(effects
-				(font
-					(size 1.27 1.27)
-				)
-			)
-		)
-		(pin "1"
-		)
-		(instances
-			(project "retroslop"
-				(path "/c091a5a9-cc18-4de7-90b1-5162a376bd78/03093195-4e98-44a3-9b51-400c2d764eeb"
-					(reference "#PWR0101")
-					(unit 1)
-				)
-			)

Commit message: tried manhattan routing
Changed lines of the file:
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@@
 		)
 	)
-	(label "~{S{2..0}}"
+	(label "~{S[2..0]}"
 		(at 52.07 121.92 0)
 		(effects

Commit message: finished routing rev3
Connections:
- net GND: now also U22.1
- net ~{RESET}: now also U2.8, U2.9; no longer U22.1
- net at D2.1 (K): now also U2.10; no longer U22.2
- net ~{HRQ I/O CH}: no longer names the net of R31.2, U4.4
- no-connect marks 9 -> 7
Other:
- moved on the sheet: U2C

Commit message: fixed things
Parts:
- added unit 6 of U22
Connections:
- net +5V: now also R42.1
- net ALLOW NMI: now also U22.13; no longer U2.3
- net FPU INSTL: now also R42.2
- net GND: now also J12.2 (Pin_2); no longer R42.2, U22.1
- net at U1.8: now also U22.1; no longer U2.2
- net at U22.2: now also U2.2
- new net: U2.3, U22.12
- no-connect marks 7 -> 6
Other:
- note added: "HOLDA <= S[2:0] == 0 & ~LOCK & (HRQ DMA)"
- note removed: "HOLDA <= S[2:0] == 0 & ~LOCK & (HRQ IO CH | HRQ DMA)"
- note removed: "~(~S[0] & ~S[1] & ~S[2] & ~LOCK & ~(~NOWS & ~HRQDMA)) & 1) ~(~S[0] & ~S[1] & ~S[2] & ~LOCK & (NOWS & HRQDMA)) & 1) (S[0] | S[1] | S[2] | LOCK | ~(NOWS & HRQDMA))) ~(S[0] | S[1] | S[2] | LOCK | ~NOWS | ~HRQDMA) ~S[1] & ~S[2] & ~S"
- moved on the sheet: U2A

Commit message: Upgraded speaker, esd protection, added dip sockets, adjusted routing
Parts:
- U1, U10, U2, U22, U29, U3, U37, U4: footprint Package_DIP:DIP-14_W7.62mm -> Package_DIP:DIP-14_W7.62mm_Socket
- U32: footprint Package_DIP:DIP-16_W7.62mm -> Package_DIP:DIP-16_W7.62mm_Socket
Other:
- note removed: "If there's no refresh is this even necessary?"
- moved on the sheet: R42

Commit message: final final review
Connections:
- net RESET renamed RESET BRD
Changed lines of the file:
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@@
 		)
 	)
-	(hierarchical_label "RESET"
+	(hierarchical_label "RESET BRD"
 		(shape input)
 		(at 38.1 193.04 180)

Commit message: modified schematic a little
Other:
- note removed: "Fuck this thing"
Changed lines of the file:
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@@
-		)
-	)
-	(text "Fuck this thing"
-		(exclude_from_sim no)
-		(at 22.352 14.478 0)
-		(effects
-			(font
-				(size 1.27 1.27)
-			)
 		)
 	)
