File: kicad/flag_registers.kicad_sch (KiCad schematic)
At the start: 8 parts, among them U17 74LS32, U54 74LS273, U55 74LS244

Commit message: made updates for rev2
Other:
- note added: "FLAG REG BIT 0: BANK ADDRESS 0 (R/W) BIT 1: BANK ADDRESS 1 (R/W) BIT 2: SPKR EN (R/W) BIT 3: SPKR GATE (R/W) BIT 4: PIT 2 OUT (R) BIT 5: I/O CH CK (R) BIT 6: Disable IO CK (R/W) BIT 7: Enable NMI (R/W)"
- note removed: "FLAG REG BIT 0: BANK ADDRESS 0 (R/W) BIT 1: BANK ADDRESS 1 (R/W) BIT 2: SPKR DATA (R/W) BIT 3: PIT GATE SPK (R/W) BIT 4: PIT 2 OUT (R) BIT 5: I/O CH CK (R) BIT 6: Disable IO CK (R/W) BIT 7: Enable NMI (R/W)"
Changed lines of the file:
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@@
 	(generator_version "10.0")
 	(paper "A4")
-	(text "FLAG REG\nBIT 0: BANK ADDRESS 0 (R/W)\nBIT 1: BANK ADDRESS 1 (R/W)\nBIT 2: SPKR DATA (R/W)\nBIT 3: PIT GATE SPK (R/W)\nBIT 4: PIT 2 OUT (R)\nBIT 5: I/O CH CK (R)\nBIT 6: Disable IO CK (R/W)\nBIT 7: Enable NMI   (R/W)"
+	(text "FLAG REG\nBIT 0: BANK ADDRESS 0 (R/W)\nBIT 1: BANK ADDRESS 1 (R/W)\nBIT 2: SPKR EN (R/W)\nBIT 3: SPKR GATE (R/W)\nBIT 4: PIT 2 OUT (R)\nBIT 5: I/O CH CK (R)\nBIT 6: Disable IO CK (R/W)\nBIT 7: Enable NMI   (R/W)"
 		(exclude_from_sim no)
 		(at 16.51 24.638 0)
