File: kicad/processor_and_control.kicad_sch (KiCad schematic)
At the start: 41 parts, among them U13 8284, U14 8088_Max_Mode, U15 8087, U16 8259A, U18 74LS373, U19 74LS373, U20 74LS373, U21 74LS245, U23 8288, U24 74LS10, Y2 14.318 MHz

Commit message: made updates for rev2
Parts:
- removed C5, C6: 47nF, Capacitor_SMD:C_1210_3225Metric_Pad1.33x2.70mm_HandSolder, symbol Device:C
Other:
- moved on the sheet: C47, C48
