File: kicad/timer.kicad_sch (KiCad schematic)
At the start: 15 parts, among them U25 LM386, U33 8254, U4 74LS00, U41 74LS175

Commit message: made updates for rev2
Parts:
- removed C86: 1 μF, Capacitor_SMD:C_1210_3225Metric_Pad1.33x2.70mm_HandSolder, symbol Device:C
- added R54: 4.7k Ω, Resistor_SMD:R_1206_3216Metric_Pad1.30x1.75mm_HandSolder, symbol Device:R
Connections:
- net +5V: now also R54.1
- net PIT GATE: now also R54.2
- net at VR2.2 (WIPER): now also U25.3 (+)
Other:
- moved on the sheet: VR2
Changed lines of the file:
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@@
 	)
 	(junction
+		(at 125.095 119.38)
+		(diameter 0)
+		(color 0 0 0 0)
+	)
+	(junction
 		(at 97.79 90.17)
 		(diameter 0)
@@
 	)
 	(junction
+		(at 111.76 90.17)
+		(diameter 0)
+		(color 0 0 0 0)
+	)
+	(junction
 		(at 245.11 85.09)
 		(diameter 0)
@@
 	(wire
 		(pts
+			(xy 125.095 100.33) (xy 125.095 119.38)
+		)
+		(stroke
+			(width 0)
+			(type default)
+		)
+	)
+	(wire
+		(pts
 			(xy 123.19 139.7) (xy 123.19 157.48)
 		)
@@
 	(wire
 		(pts
-			(xy 156.21 85.09) (xy 156.21 60.96)
+			(xy 160.655 85.09) (xy 160.655 60.96)
 		)
 		(stroke
@@
 	(wire
 		(pts
-			(xy 193.04 85.09) (xy 156.21 85.09)
+			(xy 193.04 85.09) (xy 160.655 85.09)
 		)
 		(stroke
@@
 	(wire
 		(pts
-			(xy 85.09 45.72) (xy 85.09 50.8)
+			(xy 192.405 58.42) (xy 198.12 58.42)
 		)
 		(stroke
@@
 	(wire
 		(pts
-			(xy 194.31 58.42) (xy 198.12 58.42)
+			(xy 85.09 45.72) (xy 85.09 50.8)
 		)
 		(stroke
@@
 	(wire
 		(pts
-			(xy 151.13 58.42) (xy 158.75 58.42)
+			(xy 125.095 119.38) (xy 163.83 119.38)
+		)
+		(stroke
+			(width 0)
+			(type default)
+		)
+	)
+	(wire
+		(pts
+			(xy 151.13 58.42) (xy 164.465 58.42)
 		)
 		(stroke
@@
 	(wire
 		(pts
+			(xy 111.76 90.17) (xy 125.095 90.17)
+		)
+		(stroke
+			(width 0)
+			(type default)
+		)
+	)
+	(wire
+		(pts
 			(xy 97.79 88.9) (xy 97.79 90.17)
 		)
@@
 	(wire
 		(pts
+			(xy 125.095 90.17) (xy 125.095 92.71)
+		)
+		(stroke
+			(width 0)
+			(type default)
+		)
+	)
+	(wire
+		(pts
 			(xy 81.28 111.76) (xy 87.63 111.76)
 		)
@@
 	(wire
 		(pts
-			(xy 156.21 60.96) (xy 158.75 60.96)
+			(xy 160.655 60.96) (xy 164.465 60.96)
 		)
 		(stroke
@@
 	(wire
 		(pts
-			(xy 107.95 119.38) (xy 163.83 119.38)
+			(xy 107.95 119.38) (xy 125.095 119.38)
 		)
 		(stroke
@@
 	)
 	(symbol
-		(lib_id "Device:C")
-		(at 190.5 58.42 90)
-		(unit 1)
-		(body_style 1)
-		(exclude_from_sim no)
-		(in_bom yes)
-		(on_board yes)
-		(in_pos_files yes)
-		(dnp no)
-		(fields_autoplaced yes)
-		(property "Reference" "C86"
-			(at 190.5 50.8 90)
-			(show_name no)
-			(do_not_autoplace no)
-			(effects
-				(font
-					(size 1.27 1.27)
-				)
-			)
-		)
-		(property "Value" "1 μF"
-			(at 190.5 53.34 90)
-			(show_name no)
-			(do_not_autoplace no)
-			(effects
-				(font
-					(size 1.27 1.27)
-				)
-			)
-		)
-		(property "Footprint" "Capacitor_SMD:C_1210_3225Metric_Pad1.33x2.70mm_HandSolder"
-			(at 194.31 57.4548 0)
-			(hide yes)
-			(show_name no)
-			(do_not_autoplace no)
-			(effects
-				(font
-					(size 1.27 1.27)
-				)
-			)
-		)
-		(property "Datasheet" ""
-			(at 190.5 58.42 0)
-			(hide yes)
-			(show_name no)
-			(do_not_autoplace no)
-			(effects
-				(font
-					(size 1.27 1.27)
-				)
-			)
-		)
-		(property "Description" "Unpolarized capacitor"
-			(at 190.5 58.42 0)
-			(hide yes)
-			(show_name no)
-			(do_not_autoplace no)
-			(effects
-				(font
-					(size 1.27 1.27)
-				)
-			)
-		)
-		(property "Sim.Type" ""
-			(at 190.5 58.42 0)
-			(hide yes)
-			(show_name no)
-			(do_not_autoplace no)
-			(effects
-				(font
-					(size 1.27 1.27)
-				)
-			)
-		)
-		(property "Sim.Device" ""
-			(at 190.5 58.42 90)
-			(hide yes)
-			(show_name no)
-			(do_not_autoplace no)
-			(effects
-				(font
-					(size 1.27 1.27)
-				)
-			)
-		)
-		(pin "2"
-		)
-		(pin "1"
-		)
-		(instances
-			(project "retroslop"
-				(path "/c091a5a9-cc18-4de7-90b1-5162a376bd78/3896baf8-6d60-4656-8860-0028d9860976"
-					(reference "C86")
-					(unit 1)
-				)
-			)
-		)
-	)
-	(symbol
 		(lib_id "power:VCC")
 		(at 203.2 39.37 0)
@@
 	)
 	(symbol
+		(lib_id "Device:R")
+		(at 125.095 96.52 0)
+		(unit 1)
+		(body_style 1)
+		(exclude_from_sim no)
+		(in_bom yes)
+		(on_board yes)
+		(in_pos_files yes)
+		(dnp no)
+		(fields_autoplaced yes)
+		(property "Reference" "R54"
+			(at 127.635 95.2499 0)
+			(show_name no)
+			(do_not_autoplace no)
+			(effects
+				(font
+					(size 1.27 1.27)
+				)
+				(justify left)
+			)
+		)
+		(property "Value" "4.7k Ω"
+			(at 127.635 97.7899 0)
+			(show_name no)
+			(do_not_autoplace no)
+			(effects
+				(font
+					(size 1.27 1.27)
+				)
+				(justify left)
+			)
+		)
+		(property "Footprint" "Resistor_SMD:R_1206_3216Metric_Pad1.30x1.75mm_HandSolder"
+			(at 123.317 96.52 90)
+			(hide yes)
+			(show_name no)
+			(do_not_autoplace no)
+			(effects
+				(font
+					(size 1.27 1.27)
+				)
+			)
+		)
+		(property "Datasheet" ""
+			(at 125.095 96.52 0)
+			(hide yes)
+			(show_name no)
+			(do_not_autoplace no)
+			(effects
+				(font
+					(size 1.27 1.27)
+				)
+			)
+		)
+		(property "Description" "Resistor"
+			(at 125.095 96.52 0)
+			(hide yes)
+			(show_name no)
+			(do_not_autoplace no)
+			(effects
+				(font
+					(size 1.27 1.27)
+				)
+			)
+		)
+		(property "Sim.Type" ""
+			(at 125.095 96.52 0)
+			(hide yes)
+			(show_name no)
+			(do_not_autoplace no)
+			(effects
+				(font
+					(size 1.27 1.27)
+				)
+			)
+		)
+		(property "Sim.Device" ""
+			(at 125.095 96.52 0)
+			(hide yes)
+			(show_name no)
+			(do_not_autoplace no)
+			(effects
+				(font
+					(size 1.27 1.27)
+				)
+			)
+		)
+		(pin "1"
+		)
+		(pin "2"
+		)
+		(instances
+			(project "retroslop"
+				(path "/c091a5a9-cc18-4de7-90b1-5162a376bd78/3896baf8-6d60-4656-8860-0028d9860976"
+					(reference "R54")
+					(unit 1)
+				)
+			)
+		)
+	)
+	(symbol
 		(lib_id "CVS-1508:CVS-1508")
 		(at 261.62 60.96 0)
@@
 	(symbol
 		(lib_id "N6L30T3N-103-3030:N6L30T3N-103-3030")
-		(at 158.75 58.42 0)
+		(at 164.465 58.42 0)
 		(unit 1)
 		(body_style 1)
@@
 		(fields_autoplaced yes)
 		(property "Reference" "VR2"
-			(at 172.72 50.8 0)
+			(at 178.435 50.8 0)
 			(show_name no)
 			(do_not_autoplace no)
@@
 		)
 		(property "Value" "N6L30T3N-103-3030"
-			(at 172.72 53.34 0)
+			(at 178.435 53.34 0)
 			(show_name no)
 			(do_not_autoplace no)
@@
 		)
 		(property "Footprint" "Library:N6L30T3N1033030"
-			(at 182.88 153.34 0)
+			(at 188.595 153.34 0)
 			(hide yes)
 			(show_name no)
@@
 		)
 		(property "Datasheet" "https://www.piher.net/wp-content/uploads/PIHER_N-6.pdf"
-			(at 182.88 253.34 0)
+			(at 188.595 253.34 0)
 			(hide yes)
 			(show_name no)
@@
 		)
 		(property "Description" "10 kOhms 0.1W, 1/10W PC Pins Through Hole Trimmer Potentiometer Carbon 1.0 Turn Top Adjustment"
-			(at 158.75 58.42 0)
+			(at 164.465 58.42 0)
 			(hide yes)
 			(show_name no)
@@
 		)
 		(property "Height" "7.6"
-			(at 182.88 453.34 0)
+			(at 188.595 453.34 0)
 			(hide yes)
 			(show_name no)
@@
 		)
 		(property "Mouser Part Number" ""
-			(at 182.88 553.34 0)
+			(at 188.595 553.34 0)
 			(hide yes)
 			(show_name no)
@@
 		)
 		(property "Mouser Price/Stock" ""
-			(at 182.88 653.34 0)
+			(at 188.595 653.34 0)
 			(hide yes)
 			(show_name no)
@@
 		)
 		(property "Manufacturer_Name" "Amphenol"
-			(at 182.88 753.34 0)
+			(at 188.595 753.34 0)
 			(hide yes)
 			(show_name no)
@@
 		)
 		(property "Manufacturer_Part_Number" "N6L30T3N-103-3030"
-			(at 182.88 853.34 0)
+			(at 188.595 853.34 0)
 			(hide yes)
 			(show_name no)
@@
 		)
 		(property "Sim.Type" ""
-			(at 158.75 58.42 0)
+			(at 164.465 58.42 0)
 			(hide yes)
 			(show_name no)
@@
 		)
 		(property "Sim.Device" ""
-			(at 158.75 58.42 0)
+			(at 164.465 58.42 0)
 			(hide yes)
 			(show_name no)
