File: kicad/uart.kicad_sch (KiCad schematic)
At the start: 9 parts, among them J5 DE9_Socket, U42 16550, U43 MAX232

Commit message: made updates for rev2
Parts:
- added Y1: ACO-xxxMHz-A, Oscillator:Oscillator_DIP-14, symbol Oscillator:ACO-xxxMHz-A
Connections:
- net +5V: now also Y1.1 (Tri-State), Y1.14 (Vcc)
- net GND: now also Y1.7 (GND)
- net CLK: no longer names the net of U42.16 (XIN)
- net CLK: now also Y1.8 (OUT)
Other:
- moved on the sheet: C52, C67, C68, C69, C72, C73, J5, U42, U43
